File: ToastSchematic.brd (EAGLE design)
At the start: 90 x 75 mm, 84 parts, among them Q1 DMN63D8LDW, Q2 DMN63D8LDW, Q3 DMN63D8LDW, Q4 DMN63D8LDW, T1 BPX81, T2 BPX81, T3 BPX81, T4 BPX81, T5 BPX81, T6 BPX81, U3 DRV8839_DSS_12, U4 DRV8839_DSS_12

Commit message: Finished Routing Board
Parts:
- moved R8 8.46 mm to (78.3, 25.8), turned to 180 degrees
- moved C_DISP 3.65 mm to (44.0, 36.1), turned to 0 degrees
- moved U4 0.18 mm to (36.8, 42.5)
Routing:
- net REC_R: track 3.22 -> 62.0 mm, vias 0 -> 4
- net REC_L: track 0.00 -> 56.6 mm, vias 0 -> 3
- net +3V3: track 40.5 -> 80.6 mm, vias 0 -> 4
- net REC_DR: track 4.93 -> 36.4 mm, vias 0 -> 6
- net REC_FR: track 2.71 -> 24.9 mm, vias 0 -> 4
- net DISP_RS: track 0.00 -> 22.0 mm, vias 0 -> 1
- net DISP_IN: track 0.00 -> 20.9 mm, vias 0 -> 2
- net REC_FL: track 0.00 -> 19.2 mm, vias 0 -> 2
- net DISP_CLK: track 0.00 -> 18.2 mm, vias 0 -> 3
- net +5V: track 104.9 -> 123.0 mm, vias 5 -> 11
- net REC_DL: track 3.82 -> 21.0 mm, vias 0 -> 2
- net BUZZER: track 6.17 -> 22.0 mm, vias 0 -> 2
- net NRST: track 73.2 -> 87.3 mm, vias 5 -> 6
- net IR_FL: track 1.86 -> 14.9 mm, vias 0 -> 2
- net N$25: track 0.00 -> 12.9 mm
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- added copper zone on layer 16, net +5V
